File: doc/layout/growbox/growbox.sch (KiCad schematic (older format))
At the start: 5 parts

Commit message: Add files via upload
Parts:
- added 10k (x4): R, symbol Device:R
- added U? (x3): DS18B20, Package_TO_SOT_THT:TO-92_Inline, symbol Sensor_Temperature:DS18B20
- added U? (x2): Luftfeuchte&Temp_DHT11, Sensor:Aosong_DHT11_5.5x12.0_P2.54mm, symbol Sensor:DHT11
Connections:
- net labels added: 0...3V, 3V, SDA, SDL, VCC3V
- wire segments 82 -> 135
Other:
- note added: "DEBO CAP-SENS\nBodenfeuchte"
- note added: "Heizung\n(interne Regelung)\n700 W"
- note added: "Netzspannung 230V"
- note added: "NodeMCU ESP8266\nJoy-IT\n"
- note added: "Real Time Clock\nZS-042\nI2C"
- note removed: "Heizung\n700 W"
- note removed: "Netz"
- note removed: "NodeMCU ESP8266\nJoy-IT\nhttps://joy-it.net/de/products/SBC-NodeMCU\n"
